File: PCB/HV.sch (KiCad schematic (older format))
At the start: 42 parts, among them J1 Barrel_Jack, J3 Conn_01x03_Male, J4 Conn_01x03_Male, Q1 MPSA42, Q2 MPSA42, Q3 MPSA42, Q4 MPSA42, U1 L7805, U10 74141, U11 74141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

Commit message: Some PCB fixes
Parts:
- added C3: 100uF, Capacitors_THT:CP_Radial_D8.0mm_P2.50mm, symbol CP
- added C4: 100nF, Capacitor_THT:C_Disc_D5.0mm_W2.5mm_P5.00mm, symbol C
- added C5, C6: 1nF, Capacitor_THT:C_Disc_D3.0mm_W1.6mm_P2.50mm, symbol C
- added C7: CP, Capacitors_THT:CP_Radial_D8.0mm_P2.50mm, symbol CP
- added D1: 1N5819, Diode_THT:D_DO-41_SOD81_P10.16mm_Horizontal, symbol 1N5819
- added D2: UF4007, Diode_THT:D_A-405_P10.16mm_Horizontal, symbol UF5400
- added J2: Conn_01x03_Male, Connectors_JST:JST_EH_B03B-EH-A_03x2.50mm_Straight, symbol Conn_01x03_Male
- added L1: 150uH, Inductor_THT:L_Radial_D12.5mm_P7.00mm_Fastron_09HCP, symbol L
- added Q5: BC516, TO_SOT_Packages_THT:TO-92_Inline_Wide, symbol BC516
- added Q6: IRF640, Package_DirectFET:DirectFET_MP, symbol IRF6637
- added R1: 0R1/1W, Resistor_THT:R_Axial_DIN0411_L9.9mm_D3.6mm_P12.70mm_Horizontal, symbol R
- added R13: 240K, Resistors_THT:R_Axial_DIN0207_L6.3mm_D2.5mm_P10.16mm_Horizontal, symbol R
- added R14: 1K6, Resistors_THT:R_Axial_DIN0207_L6.3mm_D2.5mm_P10.16mm_Horizontal, symbol R
- added R2: 1K, Resistors_THT:R_Axial_DIN0207_L6.3mm_D2.5mm_P10.16mm_Horizontal, symbol R
- added RT1: 2K, Potentiometer_THT:Potentiometer_Bourns_3296W_Vertical, symbol R_POT_TRIM
- added SW1, SW2: SW_Push_Dual, Buttons_Switches_THT:SW_PUSH-12mm, symbol SW_Push_Dual
- added U8: MC34063AP, Package_DIP:DIP-8_W7.62mm, symbol MC34063AP
- C1, C2: symbol Device1:C -> C
- J1: footprint Connectors:BARREL_JACK -> (none); symbol Connector1:Barrel_Jack -> Barrel_Jack
- J3, J4: symbol Connector1:Conn_01x03_Male -> Conn_01x03_Male
- N1, N2, N3, N4, N5, N6: symbol nixies:IN-12A -> IN-12A
- NE1, NE2, NE3, NE4: symbol Device1:Lamp_Neon -> Lamp_Neon
- Q1, Q2, Q3, Q4: symbol Transistor_BJT1:MPSA42 -> MPSA42
- R10, R11, R12, R3, R4, R5, R6, R7, R8, R9: symbol Device1:R -> R
- U1: footprint TO_SOT_Packages_THT:TO-220-3_Vertical -> (none); symbol Regulator_Linear1:L7805 -> L7805
- U10, U11, U12, U13, U14, U9: symbol 74xx_IEEE1:74141 -> 74141
- U2: symbol MCU_Module1:WeMos_D1_mini -> WeMos_D1_mini
- U3: symbol Sensor1:BME280 -> BME280
- U4, U5, U6, U7: symbol 74xx1:74HC595 -> 74HC595
Connections:
- net labels added: Vdrive
- wire segments 339 -> 365
