File: PCB/NixieClock.sch (KiCad schematic (older format))
At the start: 42 parts, among them J1 Barrel_Jack, J3 Conn_01x03_Male, J4 Conn_01x03_Male, Q1 MPSA42, Q2 MPSA42, Q3 MPSA42, Q4 MPSA42, U1 L7805, U10 74141, U11 74141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

Commit message: Updated PCB files
Parts:
- C1, C2: symbol Device1:C -> NixieClock-rescue:C-Device1
- J1: symbol Connector1:Barrel_Jack -> NixieClock-rescue:Barrel_Jack-Connector1
- J3, J4: symbol Connector1:Conn_01x03_Male -> NixieClock-rescue:Conn_01x03_Male-Connector1
- N1, N2, N3, N4, N5, N6: symbol nixies:IN-12A -> NixieClock-rescue:IN-12A-nixies
- NE1, NE2, NE3, NE4: symbol Device1:Lamp_Neon -> NixieClock-rescue:Lamp_Neon-Device1
- Q1, Q2, Q3, Q4: symbol Transistor_BJT1:MPSA42 -> NixieClock-rescue:MPSA42-Transistor_BJT1
- R10, R11, R12, R3, R4, R5, R6, R7, R8, R9: symbol Device1:R -> NixieClock-rescue:R-Device1
- U1: symbol Regulator_Linear1:L7805 -> NixieClock-rescue:L7805-Regulator_Linear1
- U10, U11, U12, U13, U14, U9: symbol 74xx_IEEE1:74141 -> NixieClock-rescue:74141-74xx_IEEE1
- U2: symbol MCU_Module1:WeMos_D1_mini -> NixieClock-rescue:WeMos_D1_mini-MCU_Module1
- U3: symbol Sensor1:BME280 -> NixieClock-rescue:BME280-Sensor1
- U4, U5, U6, U7: symbol 74xx1:74HC595 -> NixieClock-rescue:74HC595-74xx1
Changed lines of the file:
@@
 $EndDescr
 $Comp
-L nixies:IN-12A N1
+L NixieClock-rescue:IN-12A-nixies N1
 U 1 1 5D644170
 P 9350 4450
@@
 $EndComp
 $Comp
-L nixies:IN-12A N2
+L NixieClock-rescue:IN-12A-nixies N2
 U 1 1 5D64431F
 P 9350 6000
@@
 $EndComp
 $Comp
-L nixies:IN-12A N3
+L NixieClock-rescue:IN-12A-nixies N3
 U 1 1 5D644397
 P 9350 8000
@@
 $EndComp
 $Comp
-L nixies:IN-12A N4
+L NixieClock-rescue:IN-12A-nixies N4
 U 1 1 5D6443EC
 P 9350 9550
@@
 $EndComp
 $Comp
-L nixies:IN-12A N5
+L NixieClock-rescue:IN-12A-nixies N5
 U 1 1 5D644484
 P 9350 11500
@@
 $EndComp
 $Comp
-L nixies:IN-12A N6
+L NixieClock-rescue:IN-12A-nixies N6
 U 1 1 5D6444E9
 P 9350 13050
@@
 $EndComp
 $Comp
-L Device1:Lamp_Neon NE1
+L NixieClock-rescue:Lamp_Neon-Device1 NE1
 U 1 1 5D645472
 P 9300 6800
@@
 $EndComp
 $Comp
-L Device1:Lamp_Neon NE2
+L NixieClock-rescue:Lamp_Neon-Device1 NE2
 U 1 1 5D6459B9
 P 9300 7100
@@
 $EndComp
 $Comp
-L Device1:Lamp_Neon NE3
+L NixieClock-rescue:Lamp_Neon-Device1 NE3
 U 1 1 5D646523
 P 9300 10350
@@
 $EndComp
 $Comp
-L Device1:Lamp_Neon NE4
+L NixieClock-rescue:Lamp_Neon-Device1 NE4
 U 1 1 5D64662F
 P 9300 10600
@@
 $EndComp
 $Comp
-L 74xx_IEEE1:74141 U9
+L NixieClock-rescue:74141-74xx_IEEE1 U9
 U 1 1 5D647224
 P 7900 4300
@@
 $EndComp
 $Comp
-L 74xx_IEEE1:74141 U10
+L NixieClock-rescue:74141-74xx_IEEE1 U10
 U 1 1 5D647468
 P 7900 5850
@@
 $EndComp
 $Comp
-L 74xx_IEEE1:74141 U11
+L NixieClock-rescue:74141-74xx_IEEE1 U11
 U 1 1 5D6474EE
 P 7900 7850
@@
 $EndComp
 $Comp
-L 74xx_IEEE1:74141 U12
+L NixieClock-rescue:74141-74xx_IEEE1 U12
 U 1 1 5D6477BA
 P 7900 9400
@@
 $EndComp
 $Comp
-L 74xx_IEEE1:74141 U13
+L NixieClock-rescue:74141-74xx_IEEE1 U13
 U 1 1 5D647A50
 P 7900 11350
@@
 $EndComp
 $Comp
-L 74xx_IEEE1:74141 U14
+L NixieClock-rescue:74141-74xx_IEEE1 U14
 U 1 1 5D647AC5
 P 7900 12900
@@
 $EndComp
 $Comp
-L 74xx1:74HC595 U5
+L NixieClock-rescue:74HC595-74xx1 U5
 U 1 1 5D648D79
 P 6200 5050
@@
 $EndComp
 $Comp
-L 74xx1:74HC595 U6
+L NixieClock-rescue:74HC595-74xx1 U6
 U 1 1 5D64948D
 P 6200 8600
@@
 $EndComp
 $Comp
-L 74xx1:74HC595 U7
+L NixieClock-rescue:74HC595-74xx1 U7
 U 1 1 5D649583
 P 6200 12100
@@
 $EndComp
 $Comp
-L Device1:R R3
+L NixieClock-rescue:R-Device1 R3
 U 1 1 5D64B297
 P 10050 4450
@@
 $EndComp
 $Comp
-L Device1:R R4
+L NixieClock-rescue:R-Device1 R4
 U 1 1 5D64B56C
 P 10050 6000
@@
 $EndComp
 $Comp
-L Device1:R R7
+L NixieClock-rescue:R-Device1 R7
 U 1 1 5D64B628
 P 10050 8000
@@
 $EndComp
 $Comp
-L Device1:R R8
+L NixieClock-rescue:R-Device1 R8
 U 1 1 5D64B6F0
 P 10050 9550
@@
 $EndComp
 $Comp
-L Device1:R R11
+L NixieClock-rescue:R-Device1 R11
 U 1 1 5D64C15A
 P 10050 11500
@@
 $EndComp
 $Comp
-L Device1:R R12
+L NixieClock-rescue:R-Device1 R12
 U 1 1 5D64C234
 P 10050 13050
@@
 $EndComp
 $Comp
-L Device1:R R9
+L NixieClock-rescue:R-Device1 R9
 U 1 1 5D64C303
 P 10050 10350
@@
 $EndComp
 $Comp
-L Device1:R R10
+L NixieClock-rescue:R-Device1 R10
 U 1 1 5D64C3F6
 P 10050 10600
@@
 $EndComp
 $Comp
-L Device1:R R5
+L NixieClock-rescue:R-Device1 R5
 U 1 1 5D64C49F
 P 10050 6800
@@
 $EndComp
 $Comp
-L Device1:R R6
+L NixieClock-rescue:R-Device1 R6
 U 1 1 5D64C8AD
 P 10050 7100
@@
 $EndComp
 $Comp
-L MCU_Module1:WeMos_D1_mini U2
+L NixieClock-rescue:WeMos_D1_mini-MCU_Module1 U2
 U 1 1 5D656ABC
 P 2600 5100
@@
 $EndComp
 $Comp
-L Regulator_Linear1:L7805 U1
+L NixieClock-rescue:L7805-Regulator_Linear1 U1
 U 1 1 5D656F44
 P 2400 1250
@@
 $EndComp
 $Comp
-L Connector1:Barrel_Jack J1
+L NixieClock-rescue:Barrel_Jack-Connector1 J1
 U 1 1 5D657187
 P 1100 1350
@@
 $EndComp
 $Comp
-L power1:GND #PWR2
+L NixieClock-rescue:GND-power1 #PWR2
 U 1 1 5D6575F4
 P 1500 1800
@@
 $EndComp
 $Comp
-L power1:+12V #PWR1
+L NixieClock-rescue:+12V-power1 #PWR1
 U 1 1 5D65771F
 P 1500 1150
@@
 $EndComp
 $Comp
-L Device1:C C1
+L NixieClock-rescue:C-Device1 C1
 U 1 1 5D657E20
 P 1900 1500
@@
 $EndComp
 $Comp
-L Device1:C C2
+L NixieClock-rescue:C-Device1 C2
 U 1 1 5D658746
 P 2800 1500
@@
 $EndComp
 $Comp
-L power1:+5V #PWR6
+L NixieClock-rescue:+5V-power1 #PWR6
 U 1 1 5D658A91
 P 2800 1150
@@
 $EndComp
 $Comp
-L power1:+5V #PWR3
+L NixieClock-rescue:+5V-power1 #PWR3
 U 1 1 5D658FEB
 P 2500 4200
@@
 NoConn ~ 2200 5100
 $Comp
-L power1:GND #PWR4
+L NixieClock-rescue:GND-power1 #PWR4
 U 1 1 5D65932C
 P 2600 6150
@@
 NoConn ~ 3000 4600
 $Comp
-L Sensor1:BME280 U3
+L NixieClock-rescue:BME280-Sensor1 U3
 U 1 1 5D65BAAA
 P 3550 3250
@@
 $EndComp
 $Comp
-L power1:GND #PWR9
+L NixieClock-rescue:GND-power1 #PWR9
 U 1 1 5D65BEAB
 P 3450 4000
@@
 $EndComp
 $Comp
-L power1:+3.3V #PWR5
+L NixieClock-rescue:+3.3V-power1 #PWR5
 U 1 1 5D65D634
 P 2700 4200
@@
 $EndComp
 $Comp
-L power1:+3.3V #PWR8
+L NixieClock-rescue:+3.3V-power1 #PWR8
 U 1 1 5D65D9F8
 P 3450 2550
@@
 NoConn ~ 3650 3850
 $Comp
-L power1:VCC #PWR7
+L NixieClock-rescue:VCC-power1 #PWR7
 U 1 1 5D66003C
 P 3000 1150
@@
 $EndComp
 $Comp
-L power1:GND #PWR13
+L NixieClock-rescue:GND-power1 #PWR13
 U 1 1 5D660F95
 P 6200 5850
@@
 $EndComp
 $Comp
-L power1:GND #PWR15
+L NixieClock-rescue:GND-power1 #PWR15
 U 1 1 5D6611E7
 P 6200 9400
@@
 $EndComp
 $Comp
-L power1:GND #PWR17
+L NixieClock-rescue:GND-power1 #PWR17
 U 1 1 5D661E29
 P 6200 12900
@@
 $EndComp
 $Comp
-L power1:VCC #PWR12
+L NixieClock-rescue:VCC-power1 #PWR12
 U 1 1 5D66317D
 P 6200 4350
@@
 $EndComp
 $Comp
-L power1:VCC #PWR14
+L NixieClock-rescue:VCC-power1 #PWR14
 U 1 1 5D66346E
 P 6200 7900
@@
 $EndComp
 $Comp
-L power1:VCC #PWR16
+L NixieClock-rescue:VCC-power1 #PWR16
 U 1 1 5D6635B7
 P 6200 11400
@@
 $EndComp
 $Comp
-L 74xx1:74HC595 U4
+L NixieClock-rescue:74HC595-74xx1 U4
 U 1 1 5D6654F3
 P 3550 8600
@@
 $EndComp
 $Comp
-L power1:GND #PWR11
+L NixieClock-rescue:GND-power1 #PWR11
 U 1 1 5D665502
 P 3550 9400
@@
 $EndComp
 $Comp
-L power1:VCC #PWR10
+L NixieClock-rescue:VCC-power1 #PWR10
 U 1 1 5D665509
 P 3550 7900
@@
 NoConn ~ 3950 8600
 $Comp
-L Transistor_BJT1:MPSA42 Q2
+L NixieClock-rescue:MPSA42-Transistor_BJT1 Q2
 U 1 1 5D6668B3
 P 6300 6700
@@
 $EndComp
 $Comp
-L Transistor_BJT1:MPSA42 Q4
+L NixieClock-rescue:MPSA42-Transistor_BJT1 Q4
 U 1 1 5D666C2F
 P 6800 7100
@@
 $EndComp
 $Comp
-L power1:GND #PWR19
+L NixieClock-rescue:GND-power1 #PWR19
 U 1 1 5D667208
 P 6650 7450
@@
 $EndComp
 $Comp
-L Transistor_BJT1:MPSA42 Q1
+L NixieClock-rescue:MPSA42-Transistor_BJT1 Q1
 U 1 1 5D66829E
 P 6200 10300
@@
 $EndComp
 $Comp
-L Transistor_BJT1:MPSA42 Q3
+L NixieClock-rescue:MPSA42-Transistor_BJT1 Q3
 U 1 1 5D6682A4
 P 6700 10700
@@
 $EndComp
 $Comp
-L power1:GND #PWR18
+L NixieClock-rescue:GND-power1 #PWR18
 U 1 1 5D6682B1
 P 6550 11050
@@
 	1400 1250 1500 1250
 $Comp
-L power1:PWR_FLAG #FLG1
+L NixieClock-rescue:PWR_FLAG-power1 #FLG1
 U 1 1 5D66CB9A
 P 1900 1150
@@
 $EndComp
 $Comp
-L power1:PWR_FLAG #FLG2
+L NixieClock-rescue:PWR_FLAG-power1 #FLG2
 U 1 1 5D66D7D7
 P 1900 1800
@@
 $EndComp
 $Comp
-L Connector1:Conn_01x03_Male J3
+L NixieClock-rescue:Conn_01x03_Male-Connector1 J3
 U 1 1 5D6521C9
 P 4150 6050
@@
 	10350 3400 10350 3650
 $Comp
-L power1:PWR_FLAG #FLG3
+L NixieClock-rescue:PWR_FLAG-power1 #FLG3
 U 1 1 5D65A925
 P 10100 3400
@@
 $EndComp
 $Comp
-L Connector1:Conn_01x03_Male J4
+L NixieClock-rescue:Conn_01x03_Male-Connector1 J4
 U 1 1 5D65B901
 P 10450 3200
@@
 Connection ~ 10350 3650
 $Comp
-L power1:GND #PWR20
+L NixieClock-rescue:GND-power1 #PWR20
 U 1 1 5D65C3C4
 P 10550 3500
@@
 $EndComp
 $Comp
-L power1:+12V #PWR21
+L NixieClock-rescue:+12V-power1 #PWR21
 U 1 1 5D65C53F
 P 10750 3400
